File: Hardware/STM32H7_DK/STM32H7_DK.kicad_pcb (KiCad board)
At the start: 2 copper layers, 63.5 x 40.6 mm, 95 parts, among them J1 OV2640, J2 Conn_02x20_Counter_Clockwise, J3 Conn_02x20_Counter_Clockwise, J4 Conn_01x02_Male, Q1 S8550, SW1 KEY, SW2 KEY, SW3 KEY, SW4 KEY, U1 XC6206P282MR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

Commit message: H7开始布线
Parts:
- removed C23, C24: 10uF, Capacitor_SMD:C_0603_1608Metric_Pad1.08x0.95mm_HandSolder
- moved U3 25.0 mm to (119.1, 142.4), turned to -90 degrees
- moved C3 21.4 mm to (116.6, 142.1), turned to -90 degrees
- moved C1 19.3 mm to (115.1, 142.1), turned to -90 degrees
- moved C31 6.18 mm to (112.8, 119.5)
- moved C30 5.68 mm to (111.1, 119.5)
- moved C17 4.42 mm to (109.0, 142.1), turned to -90 degrees
- moved SD1 4.32 mm to (136.1, 129.5)
- moved C36 3.05 mm to (95.9, 129.8), turned to 0 degrees
- moved C38 3.05 mm to (95.9, 126.7)
- moved C19 2.81 mm to (126.2, 142.1)
- moved R11 2.81 mm to (121.7, 142.1)
- moved R8 2.81 mm to (123.2, 142.1)
- moved R9 2.81 mm to (124.7, 142.1)
- moved C10 2.21 mm to (140.3, 129.6)
- moved C15 2.21 mm to (140.3, 123.5)
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Connections:
- net /PB12 renamed /CAN_RX
- net /PB13 renamed /CAN_TX
- U3 pad 1: /GYRO_MISO -> /PB4
- U3 pad 12: /GYRO_CS -> /PD7
- U3 pad 13: /GYRO_SCK -> /PB3
- U3 pad 14: /GYRO_MOSI -> /PB5
- U3 pad 4: /GYRO_INT -> /PD6
Routing:
- net +3.3V: track 0.00 -> 52.0 mm, vias 0 -> 2
- net Net-(C16-Pad1): track 0.00 -> 48.8 mm, vias 0 -> 2
- net Net-(C15-Pad1): track 0.00 -> 46.9 mm, vias 0 -> 2
- net /DCMI_VS: track 0.00 -> 32.8 mm, vias 0 -> 2
- net /PC9: track 0.00 -> 32.3 mm, vias 0 -> 1
- net /PC8: track 0.00 -> 32.2 mm, vias 0 -> 1
- net /DCMI_D7: track 0.00 -> 31.9 mm, vias 0 -> 2
- net /PB2: track 0.00 -> 31.8 mm, vias 0 -> 2
- net /PC10: track 0.00 -> 31.0 mm, vias 0 -> 1
- net /DCMI_D6: track 0.00 -> 30.8 mm, vias 0 -> 2
- net /PC11: track 0.00 -> 30.3 mm, vias 0 -> 1
- net /DCMI_D4: track 0.00 -> 29.2 mm, vias 0 -> 2
- net /PD2: track 0.00 -> 28.5 mm, vias 0 -> 1
- net /PE11: track 0.00 -> 28.3 mm, vias 0 -> 2
- net /PC12: track 0.00 -> 28.2 mm, vias 0 -> 1
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Other:
- copper layers 2 -> 4

Commit message: 继续走线
Connections:
- net /PB3 renamed /GYRO_SCK
- net /PB4 renamed /GYRO_MISO
- net /PB5 renamed /GYRO_MOSI
- net /PD6 renamed /GYRO_INT
- net /PD7 renamed /GYRO_CS
- J2 pad 1: unconnected-(J2-Pad1) -> GND
- J2 pad 2: unconnected-(J2-Pad2) -> GND
- J2 pad 3: unconnected-(J2-Pad3) -> +5V
- J2 pad 4: unconnected-(J2-Pad4) -> +5V
- J3 pad 1: unconnected-(J3-Pad1) -> GND
- J3 pad 10: unconnected-(J3-Pad10) -> /PB14
- J3 pad 2: unconnected-(J3-Pad2) -> GND
- J3 pad 3: unconnected-(J3-Pad3) -> +3.3V
- J3 pad 4: unconnected-(J3-Pad4) -> +3.3V
- J3 pad 5: unconnected-(J3-Pad5) -> /PD9
- J3 pad 6: unconnected-(J3-Pad6) -> /PD10
- J3 pad 7: unconnected-(J3-Pad7) -> /PB15
- J3 pad 8: unconnected-(J3-Pad8) -> /PD8
Routing:
- net +3.3V: track 52.0 -> 260.1 mm, vias 2 -> 12
- net /DCMI_PCLK: track 0.00 -> 40.5 mm, vias 0 -> 2
- net /DCMI_D0: track 0.00 -> 38.0 mm, vias 0 -> 2
- net /DCMI_D1: track 0.00 -> 37.4 mm, vias 0 -> 2
- net /DCMI_D5: track 1.32 -> 38.7 mm, vias 1 -> 2
- net /PD14: track 2.74 -> 39.4 mm, vias 0 -> 2
- net /PE2: track 0.00 -> 28.8 mm, vias 0 -> 2
- net /DCMI_HS: track 0.00 -> 28.7 mm, vias 0 -> 2
- net /DCMI_D2: track 0.00 -> 26.7 mm, vias 0 -> 2
- net /DCMI_D3: track 0.00 -> 25.8 mm, vias 0 -> 2
- net /RST: track 5.91 -> 28.3 mm, vias 0 -> 2
- net /PB6: track 0.00 -> 21.9 mm, vias 0 -> 2
- net /PD9: track 0.00 -> 21.0 mm, vias 0 -> 1
- net /BOOT0: track 3.46 -> 23.7 mm, vias 0 -> 2
- net /PD10: track 0.00 -> 19.1 mm, vias 0 -> 1
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