File: Hardware/STM32H7_DK/STM32H7_DK.kicad_sch (KiCad schematic)
At the start: 95 parts, among them J1 OV2640, J2 Conn_02x20_Counter_Clockwise, J3 Conn_02x20_Counter_Clockwise, J4 Conn_01x02_Male, Q1 S8550, SW1 KEY, SW2 KEY, SW3 KEY, SW4 KEY, U1 XC6206P282MR, U2 XC6206P132MR, U3 BMI270, U4 STM32H7B0VBT6, U5 SN65HVD232, U6 SPX3819M5-L-3-3, U7 W25QXX_FLASH, X1 24M有源晶振2520, Y1 25MHz, Y2 32768

Commit message: H7开始布线
Parts:
- removed C23, C24: 10uF, Capacitor_SMD:C_0603_1608Metric_Pad1.08x0.95mm_HandSolder, symbol Device:C
Connections:
- net PB3 is gone; now on net GYRO_SCK: U4.89 (PB3)
- net PB4 is gone; now on net GYRO_MISO: U4.90 (PB4)
- net PB5 is gone; now on net GYRO_MOSI: U4.91 (PB5)
- net PD6 is gone; now on net GYRO_INT: U4.87 (PD6)
- net PD7 is gone; now on net GYRO_CS: U4.88 (PD7)
Changed lines of the file:
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@@
   (junction (at 346.71 57.15) (diameter 0) (color 0 0 0 0)
   )
-  (junction (at 243.84 185.42) (diameter 0) (color 0 0 0 0)
-  )
   (junction (at 82.55 232.41) (diameter 0) (color 0 0 0 0)
   )
@@
     (stroke (width 0) (type default) (color 0 0 0 0))
   )
+  (wire (pts (xy 199.39 57.15) (xy 205.74 57.15))
+    (stroke (width 0) (type default) (color 0 0 0 0))
+  )
   (polyline (pts (xy 397.51 129.54) (xy 342.9 129.54))
     (stroke (width 0) (type default) (color 0 0 0 0))
@@
     (stroke (width 0) (type default) (color 0 0 0 0))
   )
+  (wire (pts (xy 199.39 59.69) (xy 205.74 59.69))
+    (stroke (width 0) (type default) (color 0 0 0 0))
+  )
   (wire (pts (xy 199.39 97.79) (xy 205.74 97.79))
     (stroke (width 0) (type default) (color 0 0 0 0))
@@
     (stroke (width 0) (type default) (color 0 0 0 0))
   )
+  (wire (pts (xy 167.64 87.63) (xy 173.99 87.63))
+    (stroke (width 0) (type default) (color 0 0 0 0))
+  )
   (wire (pts (xy 256.54 64.77) (xy 256.54 67.31))
     (stroke (width 0) (type default) (color 0 0 0 0))
@@
     (stroke (width 0) (type default) (color 0 0 0 0))
   )
-  (wire (pts (xy 243.84 185.42) (xy 251.46 185.42))
-    (stroke (width 0) (type default) (color 0 0 0 0))
-  )
   (wire (pts (xy 334.01 72.39) (xy 334.01 64.77))
     (stroke (width 0) (type default) (color 0 0 0 0))
@@
     (stroke (width 0) (type default) (color 0 0 0 0))
   )
-  (wire (pts (xy 236.22 185.42) (xy 243.84 185.42))
+  (wire (pts (xy 236.22 185.42) (xy 251.46 185.42))
     (stroke (width 0) (type default) (color 0 0 0 0))
   )
@@
     (stroke (width 0) (type default) (color 0 0 0 0))
   )
+  (wire (pts (xy 167.64 92.71) (xy 173.99 92.71))
+    (stroke (width 0) (type default) (color 0 0 0 0))
+  )
   (wire (pts (xy 46.99 57.15) (xy 46.99 59.69))
     (stroke (width 0) (type default) (color 0 0 0 0))
@@
     (stroke (width 0) (type default) (color 0 0 0 0))
   )
+  (wire (pts (xy 167.64 90.17) (xy 173.99 90.17))
+    (stroke (width 0) (type default) (color 0 0 0 0))
+  )
   (wire (pts (xy 351.79 85.09) (xy 321.31 85.09))
     (stroke (width 0) (type default) (color 0 0 0 0))
@@
     (effects (font (size 1.27 1.27)) (justify left bottom))
   )
+  (label "GYRO_MOSI" (at 167.64 92.71 180)
+    (effects (font (size 1.27 1.27)) (justify right bottom))
+  )
+  (label "GYRO_INT" (at 205.74 57.15 0)
+    (effects (font (size 1.27 1.27)) (justify left bottom))
+  )
   (label "PB4" (at 173.99 90.17 180)
     (effects (font (size 1.27 1.27)) (justify right bottom))
@@
     (effects (font (size 1.27 1.27)) (justify right bottom))
   )
+  (label "GYRO_MISO" (at 167.64 90.17 180)
+    (effects (font (size 1.27 1.27)) (justify right bottom))
+  )
   (label "PC11" (at 340.36 69.85 0)
     (effects (font (size 1.27 1.27)) (justify left bottom))
@@
     (effects (font (size 1.27 1.27)) (justify left bottom))
   )
+  (label "GYRO_SCK" (at 167.64 87.63 180)
+    (effects (font (size 1.27 1.27)) (justify right bottom))
+  )
   (label "PE0" (at 199.39 85.09 0)
     (effects (font (size 1.27 1.27)) (justify left bottom))
@@
     (effects (font (size 1.27 1.27)) (justify left bottom))
   )
+  (label "GYRO_CS" (at 205.74 59.69 0)
+    (effects (font (size 1.27 1.27)) (justify left bottom))
+  )
   (label "PE8" (at 199.39 105.41 0)
     (effects (font (size 1.27 1.27)) (justify left bottom))
@@
     (pin "1")
   )
-  (symbol (lib_id "power:GND") (at 243.84 193.04 0) (unit 1)
-    (in_bom yes) (on_board yes)
-    (property "Reference" "#PWR043" (id 0) (at 243.84 199.39 0)
-      (effects (font (size 1.27 1.27)) hide)
-    )
-    (property "Value" "GND" (id 1) (at 243.84 196.85 0))
-    (property "Footprint" "" (id 2) (at 243.84 193.04 0)
-      (effects (font (size 1.27 1.27)) hide)
-    )
-    (property "Datasheet" "" (id 3) (at 243.84 193.04 0)
-      (effects (font (size 1.27 1.27)) hide)
-    )
-    (pin "1")
-  )
   (symbol (lib_id "power:GND") (at 241.3 46.99 0) (unit 1)
     (in_bom yes) (on_board yes)
@@
     (pin "1")
   )
-  (symbol (lib_id "Device:C") (at 243.84 175.26 0) (unit 1)
-    (in_bom yes) (on_board yes)
-    (property "Reference" "C23" (id 0) (at 245.11 172.72 0)
-      (effects (font (size 1.27 1.27)) (justify left))
-    )
-    (property "Value" "10uF" (id 1) (at 245.11 177.8 0)
-      (effects (font (size 1.27 1.27)) (justify left))
-    )
-    (property "Footprint" "Capacitor_SMD:C_0603_1608Metric_Pad1.08x0.95mm_HandSolder" (id 2) (at 244.8052 179.07 0)
-      (effects (font (size 1.27 1.27)) hide)
-    )
-    (property "Datasheet" "~" (id 3) (at 243.84 175.26 0)
-      (effects (font (size 1.27 1.27)) hide)
-    )
-    (pin "1")
-    (pin "2")
-  )
   (symbol (lib_id "Device:R") (at 85.09 256.54 0) (unit 1)
     (in_bom yes) (on_board yes)
@@
     (pin "1")
   )
-  (symbol (lib_id "Device:C") (at 243.84 189.23 0) (unit 1)
-    (in_bom yes) (on_board yes)
-    (property "Reference" "C24" (id 0) (at 245.11 186.69 0)
-      (effects (font (size 1.27 1.27)) (justify left))
-    )
-    (property "Value" "10uF" (id 1) (at 245.11 191.77 0)
-      (effects (font (size 1.27 1.27)) (justify left))
-    )
-    (property "Footprint" "Capacitor_SMD:C_0603_1608Metric_Pad1.08x0.95mm_HandSolder" (id 2) (at 244.8052 193.04 0)
-      (effects (font (size 1.27 1.27)) hide)
-    )
-    (property "Datasheet" "~" (id 3) (at 243.84 189.23 0)
-      (effects (font (size 1.27 1.27)) hide)
-    )
-    (pin "1")
-    (pin "2")
-  )
   (symbol (lib_id "Device:R") (at 364.49 31.75 90) (unit 1)
     (in_bom yes) (on_board yes)
@@
     (pin "2")
   )
-  (symbol (lib_id "power:GND") (at 243.84 179.07 0) (unit 1)
-    (in_bom yes) (on_board yes)
-    (property "Reference" "#PWR042" (id 0) (at 243.84 185.42 0)
-      (effects (font (size 1.27 1.27)) hide)
-    )
-    (property "Value" "GND" (id 1) (at 243.84 182.88 0))
-    (property "Footprint" "" (id 2) (at 243.84 179.07 0)
-      (effects (font (size 1.27 1.27)) hide)
-    )
-    (property "Datasheet" "" (id 3) (at 243.84 179.07 0)
-      (effects (font (size 1.27 1.27)) hide)
-    )
-    (pin "1")
-  )
   (symbol (lib_id "Device:C") (at 289.56 236.22 0) (unit 1)
     (in_bom yes) (on_board yes)
@@
       (reference "#PWR041") (unit 1) (value "GND") (footprint "")
     )
-    (path "/8a8d3be6-a649-4291-ab99-1d3a0e47bf16"
-      (reference "#PWR042") (unit 1) (value "GND") (footprint "")
-    )
-    (path "/162cd867-5e40-473e-a7b5-b4edcf6346d1"
-      (reference "#PWR043") (unit 1) (value "GND") (footprint "")
-    )
     (path "/b5818b80-06c1-4df9-9047-cab6cf8f5a47"
       (reference "#PWR044") (unit 1) (value "GND") (footprint "")
@@
       (reference "C22") (unit 1) (value "12pF") (footprint "Capacitor_SMD:C_0603_1608Metric_Pad1.08x0.95mm_HandSolder")
     )
-    (path "/38432d5a-2900-416e-87f2-47a1701ce228"
-      (reference "C23") (unit 1) (value "10uF") (footprint "Capacitor_SMD:C_0603_1608Metric_Pad1.08x0.95mm_HandSolder")
-    )
-    (path "/4a29ec1f-ae40-44a9-8b77-d150f521ee80"
-      (reference "C24") (unit 1) (value "10uF") (footprint "Capacitor_SMD:C_0603_1608Metric_Pad1.08x0.95mm_HandSolder")
-    )
     (path "/aca8b967-9468-46d8-ab2f-e66d0d8bc303"

Commit message: 继续走线
Connections:
- net +3.3V: now also J3.3 (Pin_3), J3.4 (Pin_4)
- net +5V: now also J2.3 (Pin_3), J2.4 (Pin_4)
- net GND: now also J2.1 (Pin_1), J2.2 (Pin_2), J3.1 (Pin_1), J3.2 (Pin_2)
- net PB14: now also J3.10 (Pin_10)
- net PB15: now also J3.7 (Pin_7)
- net PD10: now also J3.6 (Pin_6)
- net PD8: now also J3.8 (Pin_8)
- net PD9: now also J3.5 (Pin_5)
- no-connect marks 88 -> 75
